File: double-electronic-load.kicad_pcb (KiCad board)
At the start: 2 copper layers, 49.1 x 51.1 mm, 37 parts, among them J1 Screw_Terminal_01x02, J2 Screw_Terminal_01x02, J3 Screw_Terminal_01x02, Q1 SFP50N06, Q2 SFP50N06, U1 TL431LP, U2 LM358, U3 TL431LP

Commit message: Add revision to PCB
Other:
- board text added: "V1.0"
Changed lines of the file:
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@@
     (effects (font (size 1.5 1.5) (thickness 0.3)) (justify mirror))
+  )
+  (gr_text "V1.0" (at 83.566 94.615) (layer "B.SilkS")
+    (effects (font (size 1 1) (thickness 0.15)) (justify mirror))
   )
   (gr_text "7-9VDC" (at 99.06 86.614) (layer "B.SilkS")
