File: double-electronic-load.kicad_sch (KiCad schematic)
At the start: 37 parts, among them J1 Screw_Terminal_01x02, J2 Screw_Terminal_01x02, J3 Screw_Terminal_01x02, Q1 SFP50N06, Q2 SFP50N06, U1 TL431LP, U2 LM358, U3 TL431LP

Commit message: Minor cleanup
Parts:
- H1, H2, H3, H4: value MountingHole -> M3
- J1, J2, J3: value Screw_Terminal_01x02 -> LZ128 D-508
Changed lines of the file:
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@@
       (effects (font (size 1.27 1.27)) (justify left))
     )
-    (property "Value" "Screw_Terminal_01x02" (id 1) (at 160.02 60.9599 0)
+    (property "Value" "LZ128 D-508" (id 1) (at 160.02 60.9599 0)
       (effects (font (size 1.27 1.27)) (justify left))
     )
@@
       (effects (font (size 1.27 1.27)) (justify left))
     )
-    (property "Value" "MountingHole" (id 1) (at 199.39 46.9899 0)
+    (property "Value" "M3" (id 1) (at 199.39 46.9899 0)
       (effects (font (size 1.27 1.27)) (justify left))
     )
@@
       (effects (font (size 1.27 1.27)) (justify left))
     )
-    (property "Value" "Screw_Terminal_01x02" (id 1) (at 160.02 67.3099 0)
+    (property "Value" "LZ128 D-508" (id 1) (at 160.02 67.3099 0)
       (effects (font (size 1.27 1.27)) (justify left))
     )
@@
       (effects (font (size 1.27 1.27)) (justify left))
     )
-    (property "Value" "MountingHole" (id 1) (at 199.39 57.1499 0)
+    (property "Value" "M3" (id 1) (at 199.39 57.1499 0)
       (effects (font (size 1.27 1.27)) (justify left))
     )
@@
       (effects (font (size 1.27 1.27)) (justify left))
     )
-    (property "Value" "Screw_Terminal_01x02" (id 1) (at 160.02 54.6099 0)
+    (property "Value" "LZ128 D-508" (id 1) (at 160.02 54.6099 0)
       (effects (font (size 1.27 1.27)) (justify left))
     )
@@
       (effects (font (size 1.27 1.27)) (justify left))
     )
-    (property "Value" "MountingHole" (id 1) (at 199.39 41.9099 0)
+    (property "Value" "M3" (id 1) (at 199.39 41.9099 0)
       (effects (font (size 1.27 1.27)) (justify left))
     )
@@
       (effects (font (size 1.27 1.27)) (justify left))
     )
-    (property "Value" "MountingHole" (id 1) (at 199.39 52.0699 0)
+    (property "Value" "M3" (id 1) (at 199.39 52.0699 0)
       (effects (font (size 1.27 1.27)) (justify left))
     )
@@
     )
     (path "/f5474cc4-0705-4918-aa09-452c032f8472"
-      (reference "H1") (unit 1) (value "MountingHole") (footprint "MountingHole:MountingHole_3.2mm_M3")
+      (reference "H1") (unit 1) (value "M3") (footprint "MountingHole:MountingHole_3.2mm_M3")
     )
     (path "/28836780-d4cc-47d3-993b-873c2cc8ac62"
-      (reference "H2") (unit 1) (value "MountingHole") (footprint "MountingHole:MountingHole_3.2mm_M3")
+      (reference "H2") (unit 1) (value "M3") (footprint "MountingHole:MountingHole_3.2mm_M3")
     )
     (path "/fab1a681-d82d-40d4-b5f6-14abc5d56ee8"
-      (reference "H3") (unit 1) (value "MountingHole") (footprint "MountingHole:MountingHole_3.2mm_M3")
+      (reference "H3") (unit 1) (value "M3") (footprint "MountingHole:MountingHole_3.2mm_M3")
     )
     (path "/5e449207-59b4-4535-96f1-889ce742d90e"
-      (reference "H4") (unit 1) (value "MountingHole") (footprint "MountingHole:MountingHole_3.2mm_M3")
+      (reference "H4") (unit 1) (value "M3") (footprint "MountingHole:MountingHole_3.2mm_M3")
     )
     (path "/91fcd537-d3e6-4941-a9e6-675810d06017"
-      (reference "J1") (unit 1) (value "Screw_Terminal_01x02") (footprint "Custom_Footprints:Lianzhe_LZ128_D-508_2")
+      (reference "J1") (unit 1) (value "LZ128 D-508") (footprint "Custom_Footprints:Lianzhe_LZ128_D-508_2")
     )
     (path "/0f1ccaaf-8a8d-4fe8-81aa-46abc5bda849"
-      (reference "J2") (unit 1) (value "Screw_Terminal_01x02") (footprint "Custom_Footprints:Lianzhe_LZ128_D-508_2")
+      (reference "J2") (unit 1) (value "LZ128 D-508") (footprint "Custom_Footprints:Lianzhe_LZ128_D-508_2")
     )
     (path "/384f4a3d-2644-460b-8bfa-a1d26fabd713"
-      (reference "J3") (unit 1) (value "Screw_Terminal_01x02") (footprint "Custom_Footprints:Lianzhe_LZ128_D-508_2")
+      (reference "J3") (unit 1) (value "LZ128 D-508") (footprint "Custom_Footprints:Lianzhe_LZ128_D-508_2")
     )
     (path "/a05efe74-79bf-4c40-9013-d2638b658c4d"
